File: schematic/tape_deck_circuit.kicad_pcb (KiCad board)
At the start: 2 copper layers, 11 parts, among them J2 MIDI IN, J3 SPEED POT, U1 6N138

Commit message: Continue protoboard layout
Parts:
- added A1: Arduino_Nano_v3.x, Module:Arduino_Nano, F.Cu at (109.2, 109.2)
- added J3: POWER, Connector_PinHeader_2.54mm:PinHeader_1x03_P2.54mm_Vertical, F.Cu at (162.6, 134.6)
- added U2: MCP41HVx1, midi_tape_deck:TSSOP_Breakout, F.Cu at (129.5, 116.8)
- added U3: MCP41HVx1, midi_tape_deck:TSSOP_Breakout, F.Cu at (154.9, 116.8)
- D2: footprint Pin_Headers:Pin_Header_Straight_1x02_Pitch2.54mm -> Connector_PinHeader_2.54mm:PinHeader_1x02_P2.54mm_Vertical
- J1: renamed from J2; footprint Pin_Headers:Pin_Header_Straight_1x04_Pitch2.54mm -> Connector_PinHeader_2.54mm:PinHeader_1x04_P2.54mm_Vertical
- J2: renamed from J3; footprint Pin_Headers:Pin_Header_Straight_1x03_Pitch2.54mm -> Connector_PinHeader_2.54mm:PinHeader_1x03_P2.54mm_Vertical
- moved D2 89.9 mm to (246.4, 61.0)
- moved R2 68.9 mm to (68.6, 101.6)
- moved R1 57.7 mm to (177.8, 124.5)
- moved C1 57.4 mm to (195.6, 132.1), turned to 90 degrees
- moved J1 56.6 mm to (188.0, 127.0), turned to 90 degrees
- moved C2 56.4 mm to (193.0, 132.1), turned to 90 degrees
- moved U1 46.7 mm to (175.3, 119.4), turned to 90 degrees
- moved J2 42.6 mm to (139.7, 124.5), turned to 90 degrees
- moved D1 39.2 mm to (177.8, 121.9)
- moved C3 19.8 mm to (139.7, 99.1), turned to 90 degrees
- moved C4 11.8 mm to (165.1, 99.1), turned to 90 degrees
Routing:
- net (no net): track 0.00 -> 911.9 mm
- net GND: track 0.00 -> 449.6 mm, vias 0 -> 20
- net +5V: track 0.00 -> 434.3 mm, vias 0 -> 14
- net /SCK: track 0.00 -> 255.1 mm, vias 0 -> 8
- net /MISO: track 0.00 -> 115.4 mm, vias 0 -> 4
- net /MOSI: track 0.00 -> 109.2 mm, vias 0 -> 4
- net /MIDI_IN: track 0.00 -> 105.4 mm, vias 0 -> 2
- net /CS2: track 0.00 -> 88.0 mm, vias 0 -> 2
- net /CS1: track 0.00 -> 64.1 mm, vias 0 -> 2
- net /POT_COM: track 0.00 -> 53.3 mm, vias 0 -> 4
- net +15V: track 0.00 -> 45.7 mm, vias 0 -> 2
- net /PIN5: track 0.00 -> 40.6 mm, vias 0 -> 4
- net /DPOT_B: track 0.00 -> 35.6 mm, vias 0 -> 2
- net /DPOT_W: track 0.00 -> 30.5 mm, vias 0 -> 2
- net /DPOT_A: track 0.00 -> 30.5 mm, vias 0 -> 2
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Other:
- net class Default: trace_width 0.25 -> 2.032
