File: schematic/tape_deck_circuit.kicad_sch (KiCad schematic)
At the start: 15 parts, among them J1 MIDI IN, J2 SPEED POT, J3 POWER, U1 6N138, U2 MCP41HVx1, U3 MCP41HVx1

Commit message: Clean up schematic
Parts:
- removed U2, U3: MCP41HVx1, midi_tape_deck:TSSOP_Breakout, symbol midi_tape_deck:MCP41HVx1
- added U? (x2): MCP41HVx1, symbol midi_tape_deck:MCP41HVx1
- R2: value 1k -> 220
Connections:
- net +15V: now also U?.14 (V+), U?.14 (V+)
- net +5V: now also U?.1 (VL), U?.1 (VL), U?.7 (~{SHDN}), U?.7 (~{SHDN})
- net CS1: now also U?.3 (~{CS})
- net CS2: now also U?.3 (~{CS})
- net DPOT_A: now also U?.11 (P0B)
- net DPOT_B: now also U?.13 (P0A)
- net DPOT_W: now also U?.12 (P0W)
- net GND: now also U?.10 (V-), U?.10 (V-), U?.6 (~{WLAT}), U?.6 (~{WLAT}), U?.8 (DGND), U?.8 (DGND), U?.9 (NC), U?.9 (NC)
- net MISO: now also U?.5 (SDO), U?.5 (SDO)
- net MOSI: now also U?.4 (SDI), U?.4 (SDI)
- net POT_COM: now also U?.11 (P0B), U?.12 (P0W), U?.13 (P0A)
- net SCK: now also U?.2 (SCK), U?.2 (SCK)
